File: schematics/arduino_wiring.sch (EAGLE design)
At the start: 9 parts

Commit message: Fixed mistakes in arduino based schematics
Connections:
- net N$2: now also PROGRAMMER.D7, TARGET.PB5(SCK/PCINT5); no longer PROGRAMMER.*D5, TARGET.PB2(SS/OC1B/PCINT2)
- net N$3: now also TARGET.PB4(MISO/PCINT4); no longer TARGET.PB3(MOSI/OC2A/PCINT3)
- net N$4: now also PROGRAMMER.*D5, TARGET.PB3(MOSI/OC2A/PCINT3); no longer PROGRAMMER.D7, TARGET.PB4(MISO/PCINT4)
Other:
- note added: "OLED"
- note added: "SD-CARD"
Changed lines of the file:
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@@
 <sheet>
 <plain>
+<text x="170.18" y="-5.08" size="1.778" layer="91">SD-CARD</text>
+<text x="220.98" y="-2.54" size="1.778" layer="91">OLED</text>
 </plain>
 <instances>
@@
 <pinref part="PROGRAMMER" gate="G$1" pin="D4"/>
 <wire x1="160.02" y1="86.36" x2="175.26" y2="86.36" width="0.1524" layer="91"/>
-</segment>
-</net>
-<net name="N$2" class="0">
-<segment>
-<pinref part="TARGET" gate="1" pin="PB2(SS/OC1B/PCINT2)"/>
-<wire x1="119.38" y1="45.72" x2="154.94" y2="45.72" width="0.1524" layer="91"/>
-<wire x1="154.94" y1="45.72" x2="154.94" y2="83.82" width="0.1524" layer="91"/>
-<pinref part="PROGRAMMER" gate="G$1" pin="*D5"/>
-<wire x1="154.94" y1="83.82" x2="175.26" y2="83.82" width="0.1524" layer="91"/>
-</segment>
-</net>
-<net name="N$3" class="0">
-<segment>
-<pinref part="TARGET" gate="1" pin="PB3(MOSI/OC2A/PCINT3)"/>
-<wire x1="119.38" y1="43.18" x2="157.48" y2="43.18" width="0.1524" layer="91"/>
-<wire x1="157.48" y1="43.18" x2="157.48" y2="81.28" width="0.1524" layer="91"/>
-<pinref part="PROGRAMMER" gate="G$1" pin="*D6"/>
-<wire x1="157.48" y1="81.28" x2="175.26" y2="81.28" width="0.1524" layer="91"/>
-</segment>
-</net>
-<net name="N$4" class="0">
-<segment>
-<pinref part="TARGET" gate="1" pin="PB4(MISO/PCINT4)"/>
-<wire x1="119.38" y1="40.64" x2="160.02" y2="40.64" width="0.1524" layer="91"/>
-<pinref part="PROGRAMMER" gate="G$1" pin="D7"/>
-<wire x1="160.02" y1="40.64" x2="160.02" y2="78.74" width="0.1524" layer="91"/>
-<wire x1="160.02" y1="78.74" x2="175.26" y2="78.74" width="0.1524" layer="91"/>
 </segment>
 </net>
@@
 </segment>
 </net>
+<net name="N$2" class="0">
+<segment>
+<pinref part="PROGRAMMER" gate="G$1" pin="D7"/>
+<wire x1="175.26" y1="78.74" x2="160.02" y2="78.74" width="0.1524" layer="91"/>
+<wire x1="160.02" y1="78.74" x2="160.02" y2="38.1" width="0.1524" layer="91"/>
+<pinref part="TARGET" gate="1" pin="PB5(SCK/PCINT5)"/>
+<wire x1="160.02" y1="38.1" x2="119.38" y2="38.1" width="0.1524" layer="91"/>
+</segment>
+</net>
+<net name="N$3" class="0">
+<segment>
+<pinref part="TARGET" gate="1" pin="PB4(MISO/PCINT4)"/>
+<wire x1="119.38" y1="40.64" x2="157.48" y2="40.64" width="0.1524" layer="91"/>
+<wire x1="157.48" y1="40.64" x2="157.48" y2="81.28" width="0.1524" layer="91"/>
+<pinref part="PROGRAMMER" gate="G$1" pin="*D6"/>
+<wire x1="157.48" y1="81.28" x2="175.26" y2="81.28" width="0.1524" layer="91"/>
+</segment>
+</net>
+<net name="N$4" class="0">
+<segment>
+<pinref part="TARGET" gate="1" pin="PB3(MOSI/OC2A/PCINT3)"/>
+<wire x1="119.38" y1="43.18" x2="154.94" y2="43.18" width="0.1524" layer="91"/>
+<wire x1="154.94" y1="43.18" x2="154.94" y2="83.82" width="0.1524" layer="91"/>
+<pinref part="PROGRAMMER" gate="G$1" pin="*D5"/>
+<wire x1="154.94" y1="83.82" x2="175.26" y2="83.82" width="0.1524" layer="91"/>
+</segment>
+</net>
