File: schematics-target/pcb.brd (EAGLE design)
At the start: 49.5 x 35.2 mm, 8 parts, among them Q1 16Mhz

Commit message: Further work on target board
Parts:
- moved C2 1.27 mm to (31.8, 5.08)
- moved ISP 1.27 mm to (6.35, 6.35)
- moved R4 1.27 mm to (6.35, 14.0)
- moved C1 1.27 mm to (26.7, 5.08)
- moved C10 1.27 mm to (22.9, 15.2)
- moved C8 1.27 mm to (22.9, 33.0)
- moved Q1 1.27 mm to (29.2, 11.4)
- moved TARGET_ATMEGA328P 1.27 mm to (22.9, 24.1)
Other:
- board size 49.5 x 35.2 mm -> 43.2 x 35.2 mm
- board text added: "FOR ATMEGA328P"

Commit message: Updated part names in target PCB
Parts:
- renumbered C10 to C3, C8 to C4, R4 to R1
Changed lines of the file:
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@@
 <attribute name="SPICEPREFIX" value="C" x="64.77" y="21.59" size="1.778" layer="27" rot="R90" display="off"/>
 </element>
-<element name="C10" library="rcl" library_urn="urn:adsk.eagle:library:334" package="C0805" package3d_urn="urn:adsk.eagle:package:23617/2" value="100nF" x="22.86" y="15.24" smashed="yes" rot="R180">
+<element name="C3" library="rcl" library_urn="urn:adsk.eagle:library:334" package="C0805" package3d_urn="urn:adsk.eagle:package:23617/2" value="100nF" x="22.86" y="15.24" smashed="yes" rot="R180">
 <attribute name="NAME" x="24.13" y="13.97" size="1.27" layer="25" rot="R180"/>
 <attribute name="POPULARITY" value="88" x="-22.86" y="41.91" size="1.778" layer="27" rot="R180" display="off"/>
@@
 <attribute name="SPICEPREFIX" value="C" x="69.85" y="27.94" size="1.778" layer="27" rot="R90" display="off"/>
 </element>
-<element name="C8" library="rcl" library_urn="urn:adsk.eagle:library:334" package="C0805" package3d_urn="urn:adsk.eagle:package:23617/2" value="100nF" x="22.86" y="33.02" smashed="yes" rot="R180">
+<element name="C4" library="rcl" library_urn="urn:adsk.eagle:library:334" package="C0805" package3d_urn="urn:adsk.eagle:package:23617/2" value="100nF" x="22.86" y="33.02" smashed="yes" rot="R180">
 <attribute name="NAME" x="24.13" y="31.75" size="1.27" layer="25" rot="R180"/>
 <attribute name="POPULARITY" value="88" x="-16.51" y="59.69" size="1.778" layer="27" rot="R180" display="off"/>
@@
 <attribute name="POPULARITY" value="59" x="0" y="39.37" size="1.778" layer="27" rot="R180" display="off"/>
 </element>
-<element name="R4" library="rcl" library_urn="urn:adsk.eagle:library:334" package="R0805" package3d_urn="urn:adsk.eagle:package:23553/2" value="10k" x="6.35" y="13.97" smashed="yes" rot="R90">
+<element name="R1" library="rcl" library_urn="urn:adsk.eagle:library:334" package="R0805" package3d_urn="urn:adsk.eagle:package:23553/2" value="10k" x="6.35" y="13.97" smashed="yes" rot="R90">
 <attribute name="NAME" x="7.62" y="14.605" size="1.27" layer="25" rot="R270"/>
 <attribute name="POPULARITY" value="86" x="44.45" y="41.91" size="1.778" layer="27" rot="R90" display="off"/>
@@
 <contactref element="C1" pad="1"/>
 <contactref element="C2" pad="1"/>
-<contactref element="C8" pad="2"/>
+<contactref element="C4" pad="2"/>
 <contactref element="TARGET_ATMEGA328P" pad="8"/>
 <contactref element="TARGET_ATMEGA328P" pad="22"/>
-<contactref element="C10" pad="1"/>
+<contactref element="C3" pad="1"/>
 <contactref element="ISP" pad="6"/>
 <wire x1="21.91" y1="33.02" x2="21.59" y2="32.7" width="0.508" layer="1"/>
@@
 </signal>
 <signal name="+5V" class="1">
-<contactref element="R4" pad="1"/>
+<contactref element="R1" pad="1"/>
 <contactref element="TARGET_ATMEGA328P" pad="7"/>
 <contactref element="TARGET_ATMEGA328P" pad="20"/>
-<contactref element="C10" pad="2"/>
+<contactref element="C3" pad="2"/>
 <contactref element="ISP" pad="2"/>
 <wire x1="21.59" y1="20.32" x2="21.59" y2="15.24" width="0.508" layer="1"/>
@@
 </signal>
 <signal name="RESET">
-<contactref element="R4" pad="2"/>
+<contactref element="R1" pad="2"/>
 <contactref element="TARGET_ATMEGA328P" pad="1"/>
 <contactref element="ISP" pad="5"/>
@@
 </signal>
 <signal name="N$22">
-<contactref element="C8" pad="1"/>
+<contactref element="C4" pad="1"/>
 <contactref element="TARGET_ATMEGA328P" pad="21"/>
 <wire x1="23.81" y1="33.02" x2="24.13" y2="32.7" width="0.508" layer="1"/>
